File: aek2_usb.sch (KiCad schematic (older format))
At the start: 242 parts, among them J1 Conn_01x04, J2 Conn_01x04, U1 ATmega32A-PU

Commit message: remove ISO support because layout is wrong
Parts:
- removed D108: D_Small, custom_parts:D_DO-35_SOD27_P7.62mm_Horizontal, symbol Device:D_Small
- removed MX106: MX-NoLED, Alps_Only:ALPS-1.25U, symbol MX_Alps_Hybrid:MX-NoLED
- removed MX107, MX109: MX-NoLED, Alps_Only:ALPS-1U, symbol MX_Alps_Hybrid:MX-NoLED
- removed MX108: MX-NoLED, Alps_Only:ALPS-2U, symbol MX_Alps_Hybrid:MX-NoLED
Connections:
- net col1: now also MX56.1 (COL)
- net col10: now also MX65.1 (COL); no longer MX64.1 (COL)
- net col11: no longer MX65.1 (COL)
- net col2: now also MX57.1 (COL); no longer MX56.1 (COL)
- net col3: now also MX58.1 (COL); no longer MX57.1 (COL)
- net col4: now also MX59.1 (COL); no longer MX58.1 (COL)
- net col5: now also MX60.1 (COL); no longer MX59.1 (COL)
- net col6: now also MX61.1 (COL); no longer MX60.1 (COL)
- net col7: now also MX62.1 (COL); no longer MX61.1 (COL)
- net col8: now also MX63.1 (COL); no longer MX62.1 (COL)
- net col9: now also MX64.1 (COL); no longer MX63.1 (COL)
- net iso_ent: no longer names the net of D56.2 (A), MX54.2 (ROW)
- net iso_sls: no longer names the net of D42.2 (A), MX40.2 (ROW)
- net split_shift: no longer names the net of D57.2 (A), MX55.2 (ROW)
Other:
- moved on the sheet: D58, D59, D60, D61, D62, D63, D64, D65, D66, D67, MX56, MX57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
