File: aek2_usb.kicad_pcb (KiCad board)
At the start: 2 copper layers, 439 x 141.6 mm, 246 parts, among them J1 Conn_01x04, J2 Conn_01x04, U1 ATmega32A-PU

Commit message: remove ISO support because layout is wrong
Parts:
- removed D108: D_Small, custom_parts:D_DO-35_SOD27_P7.62mm_Horizontal
- removed MX106: MX-NoLED, Alps_Only:ALPS-1.25U
- removed MX107, MX109: MX-NoLED, Alps_Only:ALPS-1U
- removed MX108: MX-NoLED, Alps_Only:ALPS-2U
- moved D57 31.6 mm to (121.4, 227.8)
- moved D56 9.22 mm to (360.0, 208.9)
- moved D42 0.85 mm to (366.4, 189.9)
Connections:
- net iso_ent renamed Net-(D56-Pad2)
- net iso_sls renamed Net-(D42-Pad2)
- net split_shift renamed Net-(D57-Pad2)
- MX56 pad 1: col2 -> col1
- MX57 pad 1: col3 -> col2
- MX58 pad 1: col4 -> col3
- MX59 pad 1: col5 -> col4
- MX60 pad 1: col6 -> col5
- MX61 pad 1: col7 -> col6
- MX62 pad 1: col8 -> col7
- MX63 pad 1: col9 -> col8
- MX64 pad 1: col10 -> col9
- MX65 pad 1: col11 -> col10
Routing:
- net Net-(D42-Pad2): track 50.5 -> 8.87 mm
- net col5: track 656.4 -> 621.0 mm
- net row4: track 362.6 -> 330.9 mm
- net col10: track 540.8 -> 517.8 mm
- net col2: track 571.2 -> 548.3 mm
- net col6: track 819.1 -> 800.0 mm
- net col7: track 842.7 -> 823.5 mm
- net col4: track 579.6 -> 560.6 mm
- net col8: track 752.7 -> 733.7 mm
- net col3: track 596.5 -> 577.5 mm
- net col9: track 659.9 -> 641.0 mm
- net col1: track 502.6 -> 485.7 mm
- net Net-(D56-Pad2): track 20.9 -> 8.23 mm
- net Net-(D57-Pad2): track 24.6 -> 12.3 mm
- net col0: track 516.3 -> 504.3 mm
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